Commit message: Added ChairInterface class files

File: src/wheel_chair/description/urdf/wheel_chair_description.urdf copy.xacro (robot description, xacro)
@@ -3,6 +3,6 @@
   <xacro:macro name="wheel_chair" params="prefix">
 <!-- Define robot constants -->
-  <xacro:property name="base_width" value="0.31"/>
-  <xacro:property name="base_length" value="0.42"/>
+  <xacro:property name="base_width" value="0.51"/>
+  <xacro:property name="base_length" value="0.62"/>
   <xacro:property name="base_height" value="0.18"/>
   <xacro:property name="wheel_radius" value="0.10"/>
